Commit message: update gazebo

File: heron_description/urdf/base.urdf.xacro (robot description, xacro)
@@ -26,5 +26,5 @@
 This program contains the description of the robot base model for the Clearpath heron
 -->
-<robot
+<robot name="heron"
     xmlns:xi="http://www.w3.org/2001/XInclude"
     xmlns:gazebo="http://playerstage.sourceforge.net/gazebo/xmlschema/#gz"
@@ -39,5 +39,5 @@
     xmlns:renderable="http://playerstage.sourceforge.net/gazebo/xmlschema/#renderable"
     xmlns:physics="http://playerstage.sourceforge.net/gazebo/xmlschema/#physics"
-    xmlns:xacro="http://ros.org/wiki/xacro" name="heron">
+    xmlns:xacro="http://ros.org/wiki/xacro" >
     <!-- Included URDF/XACRO Files -->
     <xacro:include filename="$(find heron_description)/urdf/materials.urdf.xacro" />
@@ -45,5 +45,80 @@
     <!-- PROPERTY LIST -->
     <!--All units in m-kg-s-radians unit system -->
-    <property name="M_PI" value="3.1415926535897931" />
+    <xacro:property name="M_PI" value="3.1415926535897931" />
+    <xacro:property name="x_com" value="0.00000000" /> <!-- com : center of mass -->
+    <xacro:property name="y_com" value="0.00000000" /> <!-- com : center of mass -->
+    <xacro:property name="z_com" value="0.00000000" /> <!-- com : center of mass -->
+    <xacro:property name="x_size" value="1.0" />
+    <xacro:property name="y_size" value="1.0" />
+    <xacro:property name="z_size" value="1.0" />
+    <xacro:property name="mass" value="0.1" /> <!-- in kg-->
+    <xacro:property name="ixx_com_cs" value="0.01" /> <!-- at center of mass aligned with coordinate system, kg*m^2-->
+    <xacro:property name="ixy_com_cs" value="0.0" /> <!-- at center of mass aligned with coordinate system, kg*m^2-->
+    <xacro:property name="ixz_com_cs" value="0.0" /> <!-- at center of mass aligned with coordinate system, kg*m^2-->
+    <xacro:property name="iyy_com_cs" value="0.01" /> <!-- at center of mass aligned with coordinate system, kg*m^2-->
+    <xacro:property name="iyz_com_cs" value="0.00" /> <!-- at center of mass aligned with coordinate system, kg*m^2-->
+    <xacro:property name="izz_com_cs" value="0.01" /> <!-- at center of mass aligned with coordinate system, kg*m^2-->
+    <!-- heron part macro -->
+    <xacro:macro name="heron_part" params="parent name mesh translateX translateY translateZ rotateX rotateY rotateZ color">
+        <joint name="${parent}_${name}_joint" type="fixed">
+            <origin xyz="${translateX} ${translateY} ${translateZ}"
+                rpy="${rotateX} ${rotateY} ${rotateZ}" />
+            <parent link="${parent}" />
+            <child link="${parent}_${name}_part" />
+        </joint>
+        <link name="${parent}_${name}_part">
+            <inertial>
+                <mass value="${mass}" />
+                <origin xyz="${x_com} ${y_com} ${z_com}" />
+                <inertia ixx="${ixx_com_cs}" ixy="${ixy_com_cs}" ixz="${ixz_com_cs}"
+                    iyy="${iyy_com_cs}" iyz="${iyz_com_cs}" izz="${izz_com_cs}" />
+            </inertial>
+            <visual>
+                <origin xyz="0 0 0" rpy="0 0 0" />
+                <geometry>
+                    <mesh filename="package://heron_description/meshes/${mesh}.stl" />
+                </geometry>
+                <material name="${color}" />
+            </visual>
+            <collision>
+                <origin xyz="0 0 0" rpy="0 0 0"/>
+                <geometry>
+                    <box size="0.001 0.001 0.001" />
+                    <!--the collision boundary for parts are taken into account
+                         by collision boundary of the base_link-->
+                </geometry>
+            </collision>
+        </link>
+    </xacro:macro>
+    <!-- fake wheel part macro -->
+    <xacro:macro name="fake_wheel_part" params="parent pos1 pos2 translateX translateY translateZ rotateX rotateY rotateZ color">
+        <joint name="${pos1}_${pos2}_wheel_joint" type="continuous">
+            <axis xyz="0 1 0"/>
+            <origin xyz="${translateX} ${translateY} ${translateZ}"
+                rpy="${rotateX} ${rotateY} ${rotateZ}" />
+            <parent link="${parent}" />
+            <child link="${pos1}_${pos2}_wheel_part" />
+        </joint>
+        <link name="${pos1}_${pos2}_wheel_part">
+            <inertial>
+                <mass value="0.01" />
+                <inertia ixx="0.001" ixy="0" ixz="0"
+                    iyy="0.001" iyz="0" izz="0.001" />
+            </inertial>
+            <visual>
+                <origin xyz="0 0 0" rpy="0 ${M_PI/2} 0"/>
+                <geometry>
+                    <cylinder length="0.01" radius="0.05" />
+                </geometry>
+                <material name="${color}" />
+            </visual>
+            <collision>
+                <origin xyz="0 0 0" rpy="0 ${M_PI/2} 0"/>
+                <geometry>
+                    <cylinder length="0.01" radius="0.05" />
+                </geometry>
+            </collision>
+        </link>
+    </xacro:macro>
     <!-- BASE-FOOTPRINT -->
     <!-- base_footprint is a fictitious link(frame) that is on the ground right below base_link origin, navigation stack depends on this frame -->
@@ -67,5 +142,5 @@
     </gazebo>
     <joint name="base_footprint_joint" type="fixed">
-    <origin xyz="0 0 0" rpy="0 0 0" />
+        <origin xyz="0 0 0" rpy="0 0 0" />
         <parent link="base_footprint"/>
         <child link="base_link" />
@@ -76,7 +151,12 @@
         <inertial>
             <mass value="29" />
-            <!--This is the pose of the inertial reference frame, relative to the link reference frame. The origin of the inertial reference frame needs to be at the center of gravity. The axes of the inertial reference frame do not need to be aligned with the principal axes of the inertia.-->
+            <!--This is the pose of the inertial reference frame, relative to the link reference frame.
+                 The origin of the inertial reference frame needs to be at the center of gravity.
+                 The axes of the inertial reference frame do not need to be aligned with the principal axes of the inertia.-->
             <origin xyz="0 0 0" />
-            <!--The 3x3 rotational inertia matrix. Because the rotational inertia matrix is symmetric, only 6 above-diagonal elements of this matrix are specified here, using the attributes ixx, ixy, ixz, iyy, iyz, izz.-->
+            <!--The 3x3 rotational inertia matrix.
+                 Because the rotational inertia matrix is symmetric,
+                 only 6 above-diagonal elements of this matrix are specified here,
+                 using the attributes ixx, ixy, ixz, iyy, iyz, izz.-->
             <inertia ixx="10" ixy="0" ixz="0" iyy="10" iyz="0" izz="10" />
         </inertial>
@@ -89,7 +169,8 @@
         </visual>
         <collision>
-          <origin xyz="0 0 0" rpy="0 0 0" />
-          <geometry>
-                <box size = "0.1 0.1 0.1"/> <!--making it slightly bigger in x and z direction-->
+            <origin xyz="0 0 0" rpy="0 0 0" />
+            <geometry>
+                <box size = "0.1 0.1 0.1"/>
+                <!--making it slightly bigger in x and z direction-->
             </geometry>
         </collision>
@@ -101,18 +182,35 @@
     <!-- PANEL-LINKS -->
     <!-- Top Plate -->
-    <heron_part parent="base_footprint" name="left_panel" mesh="left_panel"
-          translateX="0.0" translateY="-0.35" translateZ="0.05"
-          rotateX="${M_PI/2}" rotateY="0.0" rotateZ="${M_PI/2}"
-          color="Yellow" />
+    <xacro:heron_part parent="base_footprint" name="left_panel" mesh="left_panel"
+        translateX="0.0" translateY="-0.35" translateZ="0.05"
+        rotateX="${M_PI/2}" rotateY="0.0" rotateZ="${M_PI/2}"
+        color="Yellow" />
     <gazebo reference="base_footprint_left_panel_part">
         <material>Gazebo/Yellow</material>
     </gazebo>
-    <heron_part parent="base_footprint" name="right_panel" mesh="right_panel"
-          translateX="0.0" translateY="0.35" translateZ="0.05"
-          rotateX="${M_PI/2}" rotateY="0.0" rotateZ="${-M_PI/2}"
-          color="Yellow" />
+    <xacro:heron_part parent="base_footprint" name="right_panel" mesh="right_panel"
+        translateX="0.0" translateY="0.35" translateZ="0.05"
+        rotateX="${M_PI/2}" rotateY="0.0" rotateZ="${-M_PI/2}"
+        color="Yellow" />
     <gazebo reference="base_footprint_right_panel_part">
         <material>Gazebo/Yellow</material>
     </gazebo>
+    <!--fake wheels
+    <xacro:fake_wheel_part parent="base_footprint_left_panel_part" pos1="front" pos2="left"
+        translateX="0" translateY="0.35" translateZ="-0.5"
+        rotateX="0" rotateY="0.0" rotateZ="0.0"
+        color="White" />
+    <xacro:fake_wheel_part parent="base_footprint_left_panel_part" pos1="back" pos2="left"
+        translateX="0" translateY="-0.35" translateZ="-0.5"
+        rotateX="0" rotateY="0.0" rotateZ="0.0"
+        color="White" />
+    <xacro:fake_wheel_part parent="base_footprint_right_panel_part" pos1="front" pos2="right"
+        translateX="0" translateY="0.35" translateZ="-0.5"
+        rotateX="0" rotateY="0.0" rotateZ="0.0"
+        color="White" />
+    <xacro:fake_wheel_part parent="base_footprint_right_panel_part" pos1="back" pos2="right"
+        translateX="0" translateY="-0.35" translateZ="-0.5"
+        rotateX="0" rotateY="0.0" rotateZ="0.0"
+        color="White" /> -->
     <!--Gazebo Plugin for simulating heron dynamics,
          currently not able to hack

File: heron_description/urdf/parts.urdf.xacro (robot description, xacro)
@@ -29,49 +29,126 @@
 incorporate collision.
 -->
-<robot xmlns:sensor="http://playerstage.sourceforge.net/gazebo/xmlschema/#sensor"
-	xmlns:controller="http://playerstage.sourceforge.net/gazebo/xmlschema/#controller"
-	xmlns:interface="http://playerstage.sourceforge.net/gazebo/xmlschema/#interface"
-	xmlns:xacro="http://ros.org/wiki/xacro" name="heron_part">
-	<property name="x_com" value="0.00000000" /> <!-- com : center of mass -->
-	<property name="y_com" value="0.00000000" /> <!-- com : center of mass -->
-	<property name="z_com" value="0.00000000" /> <!-- com : center of mass -->
-	<property name="x_size" value="1.0" />
-	<property name="y_size" value="1.0" />
-	<property name="z_size" value="1.0" />
-	<property name="mass" value="0.1" /> <!-- in kg-->
-	<property name="ixx_com_cs" value="0.01" /> <!-- at center of mass aligned with coordinate system, kg*m^2-->
-	<property name="ixy_com_cs" value="0.0" /> <!-- at center of mass aligned with coordinate system, kg*m^2-->
-	<property name="ixz_com_cs" value="0.0" /> <!-- at center of mass aligned with coordinate system, kg*m^2-->
-	<property name="iyy_com_cs" value="0.01" /> <!-- at center of mass aligned with coordinate system, kg*m^2-->
-	<property name="iyz_com_cs" value="0.00" /> <!-- at center of mass aligned with coordinate system, kg*m^2-->
-	<property name="izz_com_cs" value="0.01" /> <!-- at center of mass aligned with coordinate system, kg*m^2-->
-	<xacro:macro name="heron_part" params="parent name mesh translateX translateY translateZ rotateX rotateY rotateZ color">
-		<joint name="${parent}_${name}_joint" type="fixed">
-		    <origin xyz="${translateX} ${translateY} ${translateZ}"
-		            rpy="${rotateX} ${rotateY} ${rotateZ}" />
-		    <parent link="${parent}" />
-		    <child link="${parent}_${name}_part" />
-		</joint>
-		<link name="${parent}_${name}_part">
-			<inertial>
-				<mass value="${mass}" />
-				<origin xyz="${x_com} ${y_com} ${z_com}" />
-				<inertia ixx="${ixx_com_cs}" ixy="${ixy_com_cs}" ixz="${ixz_com_cs}"
-					iyy="${iyy_com_cs}" iyz="${iyz_com_cs}" izz="${izz_com_cs}" />
-			</inertial>
-			<visual>
-				<origin xyz="0 0 0" rpy="0 0 0" />
-				<geometry>
-					<mesh filename="package://heron_description/meshes/${mesh}.stl" />
-				</geometry>
-        <material name="${color}" />
-			</visual>
-			<collision>
-				<origin xyz="0 0 0" rpy="0 0 0"/>
-				<geometry>
-					<box size="0.001 0.001 0.001" /> <!--the collision boundary for parts are taken into account by collision boundary of the base_link-->
-				</geometry>
-			</collision>
-		</link>
-  	</xacro:macro>
+<robot name="heron_sensors"
+    xmlns:xacro="http://ros.org/wiki/xacro" >
+    <xacro:property name="M_PI" value="3.1415926535897931" />
+    <!-- kinect camera -->
+    <joint name="kinect_camera_joint" type="fixed">
+        <!--<xacro:insert_block name="origin" />-->
+        <origin xyz="-0.1 -0.1 0.15" rpy="0 0 0" />
+        <parent link="base_link"/>
+        <child link="kinect_camera_link"/>
+    </joint>
+    <link name="kinect_camera_link">
+        <xacro:inertial_sphere mass="0.01" diameter="0.07" />
+        <visual>
+            <origin xyz="0 0 0" rpy="0 0 0" />
+            <geometry>
+                <mesh filename="package://hector_sensors_description/meshes/kinect_camera/kinect_camera_simple.dae"/>
+            </geometry>
+        </visual>
+        <collision>
+            <origin xyz="0 0 0" rpy="0 0 0" />
+            <geometry>
+                <mesh filename="package://hector_sensors_description/meshes/kinect_camera/kinect_camera_simple.stl"/>
+            </geometry>
+        </collision>
+    </link>
+    <joint name="kinect_camera_depth_joint" type="fixed">
+        <origin xyz="0.0 -0.02 0.0" rpy="0 0 0" />
+        <parent link="kinect_camera_link" />
+        <child link="kinect_camera_depth_frame"/>
+    </joint>
+    <link name="kinect_camera_depth_frame"/>
+    <joint name="kinect_camera_depth_optical_joint" type="fixed">
+        <origin xyz="0 0 0" rpy="${-M_PI/2} 0.0 ${-M_PI/2}" />
+        <parent link="kinect_camera_depth_frame" />
+        <child link="kinect_camera_depth_optical_frame"/>
+    </joint>
+    <link name="kinect_camera_depth_optical_frame"/>
+    <joint name="kinect_camera_rgb_joint" type="fixed">
+        <origin xyz="0.0 -0.0125 0.0" rpy="0 0 0" />
+        <parent link="kinect_camera_link" />
+        <child link="kinect_camera_rgb_frame"/>
+    </joint>
+    <link name="kinect_camera_rgb_frame"/>
+    <joint name="kinect_camera_rgb_optical_joint" type="fixed">
+        <origin xyz="0 0 0" rpy="${-M_PI/2} 0.0 ${-M_PI/2}" />
+        <parent link="kinect_camera_rgb_frame" />
+        <child link="kinect_camera_rgb_optical_frame"/>
+    </joint>
+    <link name="kinect_camera_rgb_optical_frame"/>
+    <!-- Set up camera linkage and configuration -->
+    <joint name="camera_joint" type="fixed">
+        <origin xyz="0.25 0.1 0.1" rpy="0 0 0" />
+        <parent link="base_link"/>
+        <child link="camera_link" />
+    </joint>
+    <link name="camera_link">
+        <collision>
+            <origin xyz="0 0 0" rpy="0 0 0"/>
+            <geometry>
+                <box size="0.02 0.02 0.02" />
+            </geometry>
+        </collision>
+        <visual>
+            <origin xyz="0 0 0" rpy="0 0 0"/>
+            <geometry>
+                <box size="0.02 0.02 0.02" />
+            </geometry>
+            <material name="Yellow"/>
+        </visual>
+    </link>
+    <xacro:if value="$(arg sonar_enabled)">
+        <!-- Set up sonar linkage and configuration -->
+        <joint name="base_link_sonar_link_joint" type="fixed">
+            <origin xyz="0 0 -0.1" rpy="0 1.57 0" />
+            <parent link="base_link"/>
+            <child link="sonar_link" />
+        </joint>
+        <link name="sonar_link">
+            <inertial>
+                <mass value="1"/>
+                <origin xyz="0 0 0"/>
+                <inertia ixx="0.1" ixy="0.0" ixz="0.0" iyy="0.1" iyz="0.0" izz="0.1"/>
+            </inertial>
+            <visual>
+                <origin xyz="0 0 0" rpy="0 0 0" />
+                <geometry>
+                    <mesh filename="package://hector_sensors_description/meshes/sonar_sensor/max_sonar_ez4.dae"/>
+                </geometry>
+            </visual>
+            <collision>
+                <origin xyz="0 0 0" rpy="0 0 0" />
+                <geometry>
+                    <box size="0.02 0.02 0.02" />
+                </geometry>
+            </collision>
+        </link>
+    </xacro:if>
+    <joint name="hokuyo_joint" type="fixed">
+        <axis xyz="0 1 0" />
+        <origin xyz="0.2 0.15 0.15" rpy="0 0 0"/>
+        <parent link="base_link"/>
+        <child link="hokuyo_link"/>
+    </joint>
+    <!-- Hokuyo Laser -->
+    <link name="hokuyo_link">
+        <collision>
+            <origin xyz="0 0 -0.0115" rpy="0 0 0"/>
+            <geometry>
+                <box size="0.058 0.058 0.087"/>
+            </geometry>
+        </collision>
+        <visual>
+            <origin xyz="0 0 0" rpy="0 0 0"/>
+            <geometry>
+                <mesh filename="package://hector_sensors_description/meshes/hokuyo_utm30lx/hokuyo_utm_30lx.dae"/>
+            </geometry>
+        </visual>
+        <inertial>
+            <mass value="0.27" />
+            <origin xyz="0 0 0" rpy="0 0 0"/>
+            <inertia ixx="2.632e-4" ixy="0" ixz="0" iyy="2.632e-4" iyz="0" izz="1.62e-4" />
+        </inertial>
+    </link>
 </robot>
