Commit message: update gazebo

File: heron_description/urdf/standard.urdf.xacro (robot description, xacro)
@@ -38,30 +38,34 @@
         </plugin>
     </gazebo>
-    <!-- Set up camera linkage and configuration -->
-    <joint name="base_link_camera_link_joint" type="fixed">
-		<origin xyz="0 0 0.2" rpy="0 0 0" />
-        <parent link="base_link"/>
-        <child link="camera_link" />
-    </joint>
-    <link name="camera_link">
-        <collision>
-      <origin xyz="0 0 0" rpy="0 0 0"/>
-      <geometry>
-    <box size="0.05 0.05 0.05"/>
-      </geometry>
-    </collision>
-    <visual>
-      <origin xyz="0 0 0" rpy="0 0 0"/>
-      <geometry>
-    <box size="0.05 0.05 0.05"/>
-      </geometry>
-      <material name="red"/>
-    </visual>
-        <inertial>
-            <mass value="1"/>
-            <origin xyz="0 0 0"/>
-            <inertia ixx="0.1" ixy="0.0" ixz="0.0" iyy="0.1" iyz="0.0" izz="0.1"/>
-        </inertial>
-    </link>
+    <!-- Set up kinect configuration -->
+    <gazebo reference="kinect_camera_depth_frame">
+        <sensor type="depth" name="kinect_camera">
+            <update_rate>20</update_rate>
+            <camera>
+                <horizontal_fov>${60 * M_PI/180.0}</horizontal_fov>
+                <image>
+                    <format>R8G8B8</format>
+                    <width>640</width>
+                    <height>480</height>
+                </image>
+                <clip>
+                    <near>0.05</near>
+                    <far>3</far>
+                </clip>
+            </camera>
+            <plugin name="kinect_camera_controller" filename="libgazebo_ros_openni_kinect.so">
+                <cameraName>heron/kinect_camera</cameraName>
+                <imageTopicName>rgb/image_raw</imageTopicName>
+                <cameraInfoTopicName>rgb/camera_info</cameraInfoTopicName>
+                <depthImageTopicName>depth/image_raw</depthImageTopicName>
+                <depthImageCameraInfoTopicName>depth/camera_info</depthImageCameraInfoTopicName>
+                <pointCloudTopicName>depth/points</pointCloudTopicName>
+                <pointCloudCutoff>0.05</pointCloudCutoff>
+                <pointCloudCutoffMax>5</pointCloudCutoffMax>
+                <frameName>kinect_camera_depth_optical_frame</frameName>
+            </plugin>
+        </sensor>
+    </gazebo>
+    <!-- Set up camera configuration -->
     <gazebo reference="camera_link">
         <sensor type="camera" name="camera">
@@ -103,32 +107,6 @@
         </sensor>
     </gazebo>
+    <!-- Set up sonar configuration -->
     <xacro:if value="$(arg sonar_enabled)">
-        <!-- Set up sonar linkage and configuration -->
-        <joint name="base_link_sonar_link_joint" type="fixed">
-        <origin xyz="0 0 -0.2" rpy="0 1.57 0" />
-            <parent link="base_link"/>
-            <child link="sonar_link" />
-        </joint>
-        <link name="sonar_link">
-            <inertial>
-                <mass value="1"/>
-                <origin xyz="0 0 0"/>
-                <inertia ixx="0.1" ixy="0.0" ixz="0.0" iyy="0.1" iyz="0.0" izz="0.1"/>
-            </inertial>
-         <visual>
-             <origin xyz="0 0 0" rpy="0 0 0" />
-             <geometry>
-                 <box size="0.02 0.02 0.02" />
-                 <material name="green" />
-                 <!--<mesh filename="package://hector_sensors_description/meshes/sonar_sensor/max_sonar_ez4.dae"/>-->
-             </geometry>
-         </visual>
-         <collision>
-             <origin xyz="0 0 0" rpy="0 0 0" />
-             <geometry>
-               <box size="0.02 0.02 0.02" />
-            </geometry>
-         </collision>
-        </link>
         <gazebo reference="sonar_link">
             <sensor type="ray" name="sonar_sensor">
@@ -162,5 +140,6 @@
                 <plugin name="heron_ros_sonar_controller" filename="libhector_gazebo_ros_sonar.so">
                     <gaussianNoise>0.005</gaussianNoise>
-                    <topicName>sonar</topicName>
+                    <bodyName>base_link</bodyName>
+                    <topicName>heron/sonar</topicName>
                     <frameId>sonar_link</frameId>
                     <offset>0</offset>
@@ -171,3 +150,65 @@
         </gazebo>
     </xacro:if>
+    <!-- Set up hokuyo configuration -->
+    <gazebo reference="hokuyo_link">
+        <sensor type="ray" name="head_hokuyo_sensor">
+            <pose>0 0 0 0 0 0</pose>
+            <always_on>true</always_on>
+            <visualize>true</visualize>
+            <update_rate>20</update_rate>
+            <ray>
+                <scan>
+                    <horizontal>
+                        <samples>720</samples>
+                        <resolution>1</resolution>
+                        <min_angle>${-M_PI/2}</min_angle>
+                        <max_angle>${M_PI/2}</max_angle>
+                    </horizontal>
+                </scan>
+                <range>
+                    <min>0.08</min>
+                    <max>30</max>
+                    <resolution>0.004</resolution>
+                </range>
+                <noise>
+                    <type>gaussian</type>
+                    <!-- Noise parameters based on published spec for Hokuyo laser
+               achieving "+-30mm" accuracy at range < 10m.  A mean of 0.0m and
+               stddev of 0.01m will put 99.7% of samples within 0.03m of the true
+               reading. -->
+          <mean>0.0</mean>
+          <stddev>0.01</stddev>
+      </noise>
+  </ray>
+  <plugin name="gazebo_ros_hokuyo_utm30lx_model_controller" filename="libgazebo_ros_laser.so">
+      <bodyName>base_link</bodyName>
+      <topicName>heron/laser/scan</topicName>
+      <frameName>hokuyo_link</frameName>
+  </plugin>
+    </sensor>
+</gazebo>
+<!-- ros_control plugin
+  <gazebo>
+      <plugin name="skid_steer_drive_controller" filename="libgazebo_ros_skid_steer_drive.so">
+          <alwaysOn>true</alwaysOn>
+          <updateRate>100.0</updateRate>
+          <leftFrontJoint>base_footprint_left_panel_joint</leftFrontJoint>
+          <rightFrontJoint>base_footprint_right_panel_joint</rightFrontJoint>
+          <leftRearJoint>base_footprint_left_panel_joint</leftRearJoint>
+          <rightRearJoint>base_footprint_right_panel_joint</rightRearJoint>
+          <wheelSeparation>0.7</wheelSeparation>
+          <wheelDiameter>0.01</wheelDiameter>
+          <torque>35</torque>
+          <broadcastTF>1</broadcastTF>
+          <odometryFrame>map</odometryFrame>
+          <commandTopic>cmd_vel</commandTopic>
+          <odometryTopic>odom</odometryTopic>
+          <robotBaseFrame>base_footprint</robotBaseFrame>
+      </plugin>
+      <plugin name="gazebo_ros_control" filename="libgazebo_ros_control.so" >
+          <robotNamespace>heron</robotNamespace>
+          <robotSimType>gazebo_ros_control/DefaultRobotHWSim</robotSimType>
+      </plugin>
+  </gazebo>
+  -->
 </robot>

Commit message: tune gazebo

File: heron_description/urdf/base.urdf.xacro (robot description, xacro)
@@ -121,4 +121,14 @@
         </link>
     </xacro:macro>
+    <!--world -->
+    <link name="world" />
+    <!--world to base footprint joint -->
+    <joint name="world_base_joint" type="floating">
+        <axis xyz="0 0 1"/>
+        <parent link="world"/>
+        <child link="base_footprint"/>
+        <origin rpy="0 0 0" xyz="0 0 0"/>
+        <dynamics damping="0.01" friction="0.01"/>
+    </joint>
     <!-- BASE-FOOTPRINT -->
     <!-- base_footprint is a fictitious link(frame) that is on the ground right below base_link origin, navigation stack depends on this frame -->

Commit message: remove world in gazebo

File: heron_description/urdf/base.urdf.xacro (robot description, xacro)
@@ -121,7 +121,6 @@
         </link>
     </xacro:macro>
-    <!--world -->
+    <!--world >
     <link name="world" />
-    <!--world to base footprint joint -->
     <joint name="world_base_joint" type="floating">
         <axis xyz="0 0 1"/>
@@ -130,5 +129,5 @@
         <origin rpy="0 0 0" xyz="0 0 0"/>
         <dynamics damping="0.01" friction="0.01"/>
-    </joint>
+    </joint-->
     <!-- BASE-FOOTPRINT -->
     <!-- base_footprint is a fictitious link(frame) that is on the ground right below base_link origin, navigation stack depends on this frame -->
@@ -224,7 +223,7 @@
         color="White" /> -->
     <!--Gazebo Plugin for simulating heron dynamics,
-         currently not able to hack
+         currently not able to hack-->
     <gazebo>
-      <plugin name="heron_dynamic" filename="libheron_gazebo_plugins.so">
+        <plugin name="heron_dynamic" filename="$(find heron_gazebo)/plugins/libkingfisher_gazebo_plugins.so">
             <maxForce>62.0</maxForce>
             <bodyName>base_link</bodyName>
@@ -235,4 +234,4 @@
             <rolPitDampingFactor>5.0</rolPitDampingFactor>
         </plugin>
-    </gazebo>-->
+    </gazebo>
 </robot>

Commit message: gazebo planar move plugin

File: heron_description/urdf/base.urdf.xacro (robot description, xacro)
@@ -151,5 +151,5 @@
     </gazebo>
     <joint name="base_footprint_joint" type="fixed">
-        <origin xyz="0 0 0" rpy="0 0 0" />
+        <origin xyz="-0.25 0 0" rpy="0 0 0" />
         <parent link="base_footprint"/>
         <child link="base_link" />

File: heron_description/urdf/standard.urdf.xacro (robot description, xacro)
@@ -188,27 +188,13 @@
     </sensor>
 </gazebo>
-<!-- ros_control plugin
-  <gazebo>
-      <plugin name="skid_steer_drive_controller" filename="libgazebo_ros_skid_steer_drive.so">
-          <alwaysOn>true</alwaysOn>
-          <updateRate>100.0</updateRate>
-          <leftFrontJoint>base_footprint_left_panel_joint</leftFrontJoint>
-          <rightFrontJoint>base_footprint_right_panel_joint</rightFrontJoint>
-          <leftRearJoint>base_footprint_left_panel_joint</leftRearJoint>
-          <rightRearJoint>base_footprint_right_panel_joint</rightRearJoint>
-          <wheelSeparation>0.7</wheelSeparation>
-          <wheelDiameter>0.01</wheelDiameter>
-          <torque>35</torque>
-          <broadcastTF>1</broadcastTF>
-          <odometryFrame>map</odometryFrame>
-          <commandTopic>cmd_vel</commandTopic>
-          <odometryTopic>odom</odometryTopic>
-          <robotBaseFrame>base_footprint</robotBaseFrame>
-      </plugin>
-      <plugin name="gazebo_ros_control" filename="libgazebo_ros_control.so" >
-          <robotNamespace>heron</robotNamespace>
-          <robotSimType>gazebo_ros_control/DefaultRobotHWSim</robotSimType>
-      </plugin>
-  </gazebo>
-  -->
+<!-- ros_control plugin /-->
+<gazebo>
+    <plugin name="object_controller" filename="libgazebo_ros_planar_move.so">
+        <commandTopic>cmd_vel</commandTopic>
+        <odometryTopic>odom</odometryTopic>
+        <odometryFrame>odom</odometryFrame>
+        <odometryRate>20.0</odometryRate>
+        <robotBaseFrame>base_footprint</robotBaseFrame>
+    </plugin>
+</gazebo>
 </robot>

Commit message: pond sim

File: heron_description/urdf/base.urdf.xacro (robot description, xacro)
@@ -223,5 +223,5 @@
         color="White" /> -->
     <!--Gazebo Plugin for simulating heron dynamics,
-         currently not able to hack-->
+         currently not able to hack>
     <gazebo>
         <plugin name="heron_dynamic" filename="$(find heron_gazebo)/plugins/libkingfisher_gazebo_plugins.so">
@@ -234,4 +234,4 @@
             <rolPitDampingFactor>5.0</rolPitDampingFactor>
         </plugin>
-    </gazebo>
+    </gazebo-->
 </robot>

File: heron_description/urdf/parts.urdf.xacro (robot description, xacro)
@@ -40,5 +40,10 @@
     </joint>
     <link name="kinect_camera_link">
-        <xacro:inertial_sphere mass="0.01" diameter="0.07" />
+        <!--xacro:inertial_sphere mass="0.01" diameter="0.07" /-->
+        <inertial>
+                <mass value="0.01" />
+                <origin xyz="0 0 0" rpy="0 0 0"/>
+                <inertia ixx="2.632e-4" ixy="0" ixz="0" iyy="2.632e-4" iyz="0" izz="1.62e-4" />
+            </inertial>
         <visual>
             <origin xyz="0 0 0" rpy="0 0 0" />

Commit message: modify urdf and gazebo launch

File: heron_description/urdf/base.urdf.xacro (robot description, xacro)
@@ -121,13 +121,4 @@
         </link>
     </xacro:macro>
-    <!--world >
-    <link name="world" />
-    <joint name="world_base_joint" type="floating">
-        <axis xyz="0 0 1"/>
-        <parent link="world"/>
-        <child link="base_footprint"/>
-        <origin rpy="0 0 0" xyz="0 0 0"/>
-        <dynamics damping="0.01" friction="0.01"/>
-    </joint-->
     <!-- BASE-FOOTPRINT -->
     <!-- base_footprint is a fictitious link(frame) that is on the ground right below base_link origin, navigation stack depends on this frame -->
@@ -191,16 +182,16 @@
     <!-- PANEL-LINKS -->
     <!-- Top Plate -->
-    <xacro:heron_part parent="base_footprint" name="left_panel" mesh="left_panel"
-        translateX="0.0" translateY="-0.35" translateZ="0.05"
+    <xacro:heron_part parent="base_link" name="left_panel" mesh="left_panel"
+        translateX="0" translateY="-0.35" translateZ="0.05"
         rotateX="${M_PI/2}" rotateY="0.0" rotateZ="${M_PI/2}"
         color="Yellow" />
-    <gazebo reference="base_footprint_left_panel_part">
+    <gazebo reference="base_link_left_panel_part">
         <material>Gazebo/Yellow</material>
     </gazebo>
-    <xacro:heron_part parent="base_footprint" name="right_panel" mesh="right_panel"
-        translateX="0.0" translateY="0.35" translateZ="0.05"
+    <xacro:heron_part parent="base_link" name="right_panel" mesh="right_panel"
+        translateX="0" translateY="0.35" translateZ="0.05"
         rotateX="${M_PI/2}" rotateY="0.0" rotateZ="${-M_PI/2}"
         color="Yellow" />
-    <gazebo reference="base_footprint_right_panel_part">
+    <gazebo reference="base_link_right_panel_part">
         <material>Gazebo/Yellow</material>
     </gazebo>

File: heron_description/urdf/parts.urdf.xacro (robot description, xacro)
@@ -35,5 +35,5 @@
     <joint name="kinect_camera_joint" type="fixed">
         <!--<xacro:insert_block name="origin" />-->
-        <origin xyz="-0.1 -0.1 0.15" rpy="0 0 0" />
+        <origin xyz="0.1 0 0.2" rpy="0 0 0" />
         <parent link="base_link"/>
         <child link="kinect_camera_link"/>
@@ -85,22 +85,21 @@
     <!-- Set up camera linkage and configuration -->
     <joint name="camera_joint" type="fixed">
-        <origin xyz="0.25 0.1 0.1" rpy="0 0 0" />
+        <origin xyz="0.35 0 0" rpy="0 0 0" />
         <parent link="base_link"/>
         <child link="camera_link" />
     </joint>
     <link name="camera_link">
+        <visual>
+            <origin xyz="0 0 0" rpy="0 0 0" />
+            <geometry>
+                <mesh filename="package://hector_sensors_description/meshes/thermaleye_camera/thermaleye_camera_hector_v2.dae"/>
+            </geometry>
+        </visual>
         <collision>
-            <origin xyz="0 0 0" rpy="0 0 0"/>
+            <origin xyz="0 0 0" rpy="0 0 0" />
             <geometry>
-                <box size="0.02 0.02 0.02" />
+                <mesh filename="package://hector_sensors_description/meshes/thermaleye_camera/thermaleye_camera_hector_v2.stl"/>
             </geometry>
         </collision>
-        <visual>
-            <origin xyz="0 0 0" rpy="0 0 0"/>
-            <geometry>
-                <box size="0.02 0.02 0.02" />
-            </geometry>
-            <material name="Yellow"/>
-        </visual>
     </link>
     <xacro:if value="$(arg sonar_enabled)">
@@ -133,5 +132,5 @@
     <joint name="hokuyo_joint" type="fixed">
         <axis xyz="0 1 0" />
-        <origin xyz="0.2 0.15 0.15" rpy="0 0 0"/>
+        <origin xyz="0.2 0.15 0.1" rpy="0 0 0"/>
         <parent link="base_link"/>
         <child link="hokuyo_link"/>
